Commit message: first commit with gripper
adding gripper test

File: urdf/amber_b1.urdf (robot description, URDF)
Before this commit: robot amber_urdf, 12 links, 11 joints
Links:
- removed link TOP_1
- added link Cover1_1, mass 0.057836049894173285; collision mesh filename=package://amber_urdf_description/meshes/Cover1_1.stl scale=0.001 0.001 0.001; visual mesh filename=package://amber_urdf_description/meshes/Cover1_1.stl scale=0.001 0.001 0.001
- added link Garm1_left_1, mass 0.04242624144126467; collision mesh filename=package://amber_urdf_description/meshes/Garm1_left_1.stl scale=0.001 0.001 0.001; visual mesh filename=package://amber_urdf_description/meshes/Garm1_left_1.stl scale=0.001 0.001 0.001
- added link Garm1_v1_1, mass 0.04242624144126467; collision mesh filename=package://amber_urdf_description/meshes/Garm1_v1_1.stl scale=0.001 0.001 0.001; visual mesh filename=package://amber_urdf_description/meshes/Garm1_v1_1.stl scale=0.001 0.001 0.001
- added link Garm2_left_1, mass 0.04152241646366915; collision mesh filename=package://amber_urdf_description/meshes/Garm2_left_1.stl scale=0.001 0.001 0.001; visual mesh filename=package://amber_urdf_description/meshes/Garm2_left_1.stl scale=0.001 0.001 0.001
- added link Garm2_v1_1, mass 0.04152241646366915; collision mesh filename=package://amber_urdf_description/meshes/Garm2_v1_1.stl scale=0.001 0.001 0.001; visual mesh filename=package://amber_urdf_description/meshes/Garm2_v1_1.stl scale=0.001 0.001 0.001
- added link Yaw_left_1, mass 0.13411633515691568; collision mesh filename=package://amber_urdf_description/meshes/Yaw_left_1.stl scale=0.001 0.001 0.001; visual mesh filename=package://amber_urdf_description/meshes/Yaw_left_1.stl scale=0.001 0.001 0.001
- added link Yaw_right_1, mass 0.13411633515691568; collision mesh filename=package://amber_urdf_description/meshes/Yaw_right_1.stl scale=0.001 0.001 0.001; visual mesh filename=package://amber_urdf_description/meshes/Yaw_right_1.stl scale=0.001 0.001 0.001
- added link gripper_head_v1_1, mass 1.3440613994784911; collision mesh filename=package://amber_urdf_description/meshes/gripper_head_v1_1.s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 scale=0.001 0.001 0.001; visual mesh filename=package://amber_urdf_description/meshes/gripper_head_v1_1.s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 scale=0.001 0.001 0.001
Joints:
- removed joint Rigid12
- added joint Rev13: type continuous, parent DOF6_LINK_1, child gripper_head_v1_1, origin xyz=-0.0 0.0255 0.127896 rpy=0 0 0, axis -0.0 0.0 -1.0
- added joint Rev14: type continuous, parent gripper_head_v1_1, child Garm1_v1_1, origin xyz=-0.004439 0.035292 0.096501 rpy=0 0 0, axis 0.984808 -0.173648 -0.0, limit lower=-0.8 upper=0.1 effort=100 velocity=6.159937255, mimic joint=Rev16 multiplier=-1.0 offset=0
- added joint Rev15: type continuous, parent gripper_head_v1_1, child Garm2_v1_1, origin xyz=-0.008507 0.012223 0.113763 rpy=0 0 0, axis 0.984808 -0.173648 -0.0, mimic joint=Rev14 multiplier=1.2 offset=0
- added joint Rev16: type revolute, parent gripper_head_v1_1, child Garm1_left_1, origin xyz=-0.016242 -0.031645 0.096501 rpy=0 0 0, axis 0.984808 -0.173648 -0.0, limit lower=-0.1 upper=0.8 effort=100 velocity=6.159937255
- added joint Rev17: type continuous, parent gripper_head_v1_1, child Garm2_left_1, origin xyz=-0.012174 -0.008576 0.113763 rpy=0 0 0, axis 0.984808 -0.173648 -0.0, mimic joint=Rev16 multiplier=1.2 offset=0
- added joint Rev18: type continuous, parent Garm1_v1_1, child Yaw_right_1, origin xyz=0.003069 -0.001598 0.06075 rpy=0 0 0, axis -0.984808 0.173648 0.0, mimic joint=Rev14 multiplier=1.533333333 offset=0
- added joint Rev20: type continuous, parent Garm1_left_1, child Yaw_left_1, origin xyz=0.003431 0.000452 0.06075 rpy=0 0 0, axis -0.984808 0.173648 0.0, mimic joint=Rev16 multiplier=1.533333333 offset=0
- added joint Rigid22: type fixed, parent gripper_head_v1_1, child Cover1_1, origin xyz=-0.027575 0.004862 0.067 rpy=0 0 0

File: urdf/amber_urdf.xacro (robot description, xacro)
@@ -224,14 +224,14 @@
   </collision>
 </link>
-<link name="TOP_1">
-  <inertial>
-    <origin rpy="0 0 0" xyz="-4.963925281376204e-07 -0.00019582783329597517 0.01611980646593192"/>
-    <mass value="0.15302388632599126"/>
-    <inertia ixx="4.6e-05" ixy="0.0" ixz="0.0" iyy="5e-05" iyz="0.0" izz="5.5e-05"/>
+<link name="gripper_head_v1_1">
+  <inertial>
+    <origin rpy="0 0 0" xyz="-0.00023127268430785794 4.0565269390425876e-05 0.06450548283852242"/>
+    <mass value="1.3440613994784911"/>
+    <inertia ixx="0.001879" ixy="-4.2e-05" ixz="-1.4e-05" iyy="0.001648" iyz="3e-06" izz="0.000816"/>
   </inertial>
   <visual>
     <origin rpy="0 0 0" xyz="0.0 -0.000504 -0.701955"/>
     <geometry>
-      <mesh filename="package://amber_urdf_description/meshes/TOP_1.stl" scale="0.001 0.001 0.001"/>
+      <mesh filename="package://amber_urdf_description/meshes/gripper_head_v1_1.stl" scale="0.001 0.001 0.001"/>
     </geometry>
     <material name="silver_default"/>
@@ -240,5 +240,145 @@
     <origin rpy="0 0 0" xyz="0.0 -0.000504 -0.701955"/>
     <geometry>
-      <mesh filename="package://amber_urdf_description/meshes/TOP_1.stl" scale="0.001 0.001 0.001"/>
+      <mesh filename="package://amber_urdf_description/meshes/gripper_head_v1_1.stl" scale="0.001 0.001 0.001"/>
+    </geometry>
+  </collision>
+</link>
+<link name="Garm1_v1_1">
+  <inertial>
+    <origin rpy="0 0 0" xyz="0.01142339286285327 0.005469675886271411 0.03332029659019209"/>
+    <mass value="0.04242624144126467"/>
+    <inertia ixx="1.9e-05" ixy="0.0" ixz="0.0" iyy="1.9e-05" iyz="2e-06" izz="3e-06"/>
+  </inertial>
+  <visual>
+    <origin rpy="0 0 0" xyz="0.004439 -0.035796 -0.798456"/>
+    <geometry>
+      <mesh filename="package://amber_urdf_description/meshes/Garm1_v1_1.stl" scale="0.001 0.001 0.001"/>
+    </geometry>
+    <material name="silver_default"/>
+  </visual>
+  <collision>
+    <origin rpy="0 0 0" xyz="0.004439 -0.035796 -0.798456"/>
+    <geometry>
+      <mesh filename="package://amber_urdf_description/meshes/Garm1_v1_1.stl" scale="0.001 0.001 0.001"/>
+    </geometry>
+  </collision>
+</link>
+<link name="Garm2_v1_1">
+  <inertial>
+    <origin rpy="0 0 0" xyz="0.011494368992215495 0.003559922438370491 0.02472036320342974"/>
+    <mass value="0.04152241646366915"/>
+    <inertia ixx="1.2e-05" ixy="1e-06" ixz="-0.0" iyy="1.6e-05" iyz="-0.0" izz="5e-06"/>
+  </inertial>
+  <visual>
+    <origin rpy="0 0 0" xyz="0.008507 -0.012727 -0.815718"/>
+    <geometry>
+      <mesh filename="package://amber_urdf_description/meshes/Garm2_v1_1.stl" scale="0.001 0.001 0.001"/>
+    </geometry>
+    <material name="silver_default"/>
+  </visual>
+  <collision>
+    <origin rpy="0 0 0" xyz="0.008507 -0.012727 -0.815718"/>
+    <geometry>
+      <mesh filename="package://amber_urdf_description/meshes/Garm2_v1_1.stl" scale="0.001 0.001 0.001"/>
+    </geometry>
+  </collision>
+</link>
+<link name="Garm1_left_1">
+  <inertial>
+    <origin rpy="0 0 0" xyz="0.00886367921658928 -0.00904741551475095 0.03332029658806501"/>
+    <mass value="0.04242624144126467"/>
+    <inertia ixx="1.9e-05" ixy="0.0" ixz="-0.0" iyy="1.9e-05" iyz="-2e-06" izz="3e-06"/>
+  </inertial>
+  <visual>
+    <origin rpy="0 0 0" xyz="0.016242 0.031141 -0.798456"/>
+    <geometry>
+      <mesh filename="package://amber_urdf_description/meshes/Garm1_left_1.stl" scale="0.001 0.001 0.001"/>
+    </geometry>
+    <material name="silver_default"/>
+  </visual>
+  <collision>
+    <origin rpy="0 0 0" xyz="0.016242 0.031141 -0.798456"/>
+    <geometry>
+      <mesh filename="package://amber_urdf_description/meshes/Garm1_left_1.stl" scale="0.001 0.001 0.001"/>
+    </geometry>
+  </collision>
+</link>
+<link name="Garm2_left_1">
+  <inertial>
+    <origin rpy="0 0 0" xyz="0.009580549289645798 -0.007276580609441009 0.024720363202603735"/>
+    <mass value="0.04152241646366915"/>
+    <inertia ixx="1.2e-05" ixy="1e-06" ixz="0.0" iyy="1.6e-05" iyz="0.0" izz="5e-06"/>
+  </inertial>
+  <visual>
+    <origin rpy="0 0 0" xyz="0.012174 0.008072 -0.815718"/>
+    <geometry>
+      <mesh filename="package://amber_urdf_description/meshes/Garm2_left_1.stl" scale="0.001 0.001 0.001"/>
+    </geometry>
+    <material name="silver_default"/>
+  </visual>
+  <collision>
+    <origin rpy="0 0 0" xyz="0.012174 0.008072 -0.815718"/>
+    <geometry>
+      <mesh filename="package://amber_urdf_description/meshes/Garm2_left_1.stl" scale="0.001 0.001 0.001"/>
+    </geometry>
+  </collision>
+</link>
+<link name="Yaw_right_1">
+  <inertial>
+    <origin rpy="0 0 0" xyz="0.003175663516676549 -0.022299866594133536 0.024771853265351917"/>
+    <mass value="0.13411633515691568"/>
+    <inertia ixx="5e-05" ixy="-1e-06" ixz="3e-06" iyy="4.4e-05" iyz="1.6e-05" izz="1.9e-05"/>
+  </inertial>
+  <visual>
+    <origin rpy="0 0 0" xyz="0.00137 -0.034198 -0.859206"/>
+    <geometry>
+      <mesh filename="package://amber_urdf_description/meshes/Yaw_right_1.stl" scale="0.001 0.001 0.001"/>
+    </geometry>
+    <material name="silver_default"/>
+  </visual>
+  <collision>
+    <origin rpy="0 0 0" xyz="0.00137 -0.034198 -0.859206"/>
+    <geometry>
+      <mesh filename="package://amber_urdf_description/meshes/Yaw_right_1.stl" scale="0.001 0.001 0.001"/>
+    </geometry>
+  </collision>
+</link>
+<link name="Yaw_left_1">
+  <inertial>
+    <origin rpy="0 0 0" xyz="0.010611408562765922 0.019868126962941598 0.024771853264752175"/>
+    <mass value="0.13411633515691568"/>
+    <inertia ixx="5e-05" ixy="-1e-06" ixz="-3e-06" iyy="4.4e-05" iyz="-1.6e-05" izz="1.9e-05"/>
+  </inertial>
+  <visual>
+    <origin rpy="0 0 0" xyz="0.012811 0.030689 -0.859206"/>
+    <geometry>
+      <mesh filename="package://amber_urdf_description/meshes/Yaw_left_1.stl" scale="0.001 0.001 0.001"/>
+    </geometry>
+    <material name="silver_default"/>
+  </visual>
+  <collision>
+    <origin rpy="0 0 0" xyz="0.012811 0.030689 -0.859206"/>
+    <geometry>
+      <mesh filename="package://amber_urdf_description/meshes/Yaw_left_1.stl" scale="0.001 0.001 0.001"/>
+    </geometry>
+  </collision>
+</link>
+<link name="Cover1_1">
+  <inertial>
+    <origin rpy="0 0 0" xyz="0.007227292155078693 -0.0012744011834956168 0.023355135145045502"/>
+    <mass value="0.057836049894173285"/>
+    <inertia ixx="3.3e-05" ixy="-4e-06" ixz="-1e-06" iyy="1.3e-05" iyz="0.0" izz="2.2e-05"/>
+  </inertial>
+  <visual>
+    <origin rpy="0 0 0" xyz="0.027575 -0.005366 -0.768955"/>
+    <geometry>
+      <mesh filename="package://amber_urdf_description/meshes/Cover1_1.stl" scale="0.001 0.001 0.001"/>
+    </geometry>
+    <material name="opaque119125137"/>
+  </visual>
+  <collision>
+    <origin rpy="0 0 0" xyz="0.027575 -0.005366 -0.768955"/>
+    <geometry>
+      <mesh filename="package://amber_urdf_description/meshes/Cover1_1.stl" scale="0.001 0.001 0.001"/>
     </geometry>
   </collision>
@@ -300,8 +440,57 @@
   <child link="DOF7_MOTOR_1"/>
 </joint>
-<joint name="Rigid12" type="fixed">
+<joint name="Rev13" type="continuous">
   <origin rpy="0 0 0" xyz="-0.0 0.0255 0.127896"/>
   <parent link="DOF6_LINK_1"/>
-  <child link="TOP_1"/>
+  <child link="gripper_head_v1_1"/>
+  <axis xyz="-0.0 0.0 -1.0"/>
+</joint>
+<joint name="Rev14" type="continuous">
+  <origin rpy="0 0 0" xyz="-0.004439 0.035292 0.096501"/>
+  <parent link="gripper_head_v1_1"/>
+  <child link="Garm1_v1_1"/>
+  <axis xyz="0.984808 -0.173648 -0.0"/>
+<limit lower="-0.8" upper="0.1" effort="100" velocity="6.159937255" />
+<mimic joint="Rev16" multiplier="-1.0" offset="0" />
+</joint>
+<joint name="Rev15" type="continuous">
+  <origin rpy="0 0 0" xyz="-0.008507 0.012223 0.113763"/>
+  <parent link="gripper_head_v1_1"/>
+  <child link="Garm2_v1_1"/>
+  <axis xyz="0.984808 -0.173648 -0.0"/>
+<mimic joint="Rev14" multiplier="1.2" offset="0" />
+</joint>
+<joint name="Rev16" type="revolute">
+  <origin rpy="0 0 0" xyz="-0.016242 -0.031645 0.096501"/>
+  <parent link="gripper_head_v1_1"/>
+  <child link="Garm1_left_1"/>
+  <axis xyz="0.984808 -0.173648 -0.0"/>
+<limit lower="-0.1" upper="0.8" effort="100" velocity="6.159937255" />
+</joint>
+<joint name="Rev17" type="continuous">
+  <origin rpy="0 0 0" xyz="-0.012174 -0.008576 0.113763"/>
+  <parent link="gripper_head_v1_1"/>
+  <child link="Garm2_left_1"/>
+  <axis xyz="0.984808 -0.173648 -0.0"/>
+<mimic joint="Rev16" multiplier="1.2" offset="0" />
+</joint>
+<joint name="Rev18" type="continuous">
+  <origin rpy="0 0 0" xyz="0.003069 -0.001598 0.06075"/>
+  <parent link="Garm1_v1_1"/>
+  <child link="Yaw_right_1"/>
+  <axis xyz="-0.984808 0.173648 0.0"/>
+<mimic joint="Rev14" multiplier="1.533333333" offset="0" />
+</joint>
+<joint name="Rev20" type="continuous">
+  <origin rpy="0 0 0" xyz="0.003431 0.000452 0.06075"/>
+  <parent link="Garm1_left_1"/>
+  <child link="Yaw_left_1"/>
+  <axis xyz="-0.984808 0.173648 0.0"/>
+<mimic joint="Rev16" multiplier="1.533333333" offset="0" />
+</joint>
+<joint name="Rigid22" type="fixed">
+  <origin rpy="0 0 0" xyz="-0.027575 0.004862 0.067"/>
+  <parent link="gripper_head_v1_1"/>
+  <child link="Cover1_1"/>
 </joint>
 </robot>

File: urdf/materials.xacro (robot description, xacro)
@@ -4,3 +4,6 @@
   <color rgba="0.700 0.700 0.700 1.000"/>
 </material>
+<material name="opaque119125137">
+  <color rgba="0.4666666666666667 0.49019607843137253 0.5372549019607843 1.0"/>
+</material>
 </robot>
